File: LN2544_2ch_CWW.kicad_pcb (KiCad board)
At the start: 2 copper layers, 22 x 28 mm, 44 parts, among them P1 Vin, P2 LED, P3 DIM, P4 NTC, U1 LN2544, U2 LN2544

Commit message: Upd
Parts:
- moved C5 7.05 mm to (110.8, 125.1), turned to 270 degrees
- moved C6 1.73 mm to (109.0, 125.1), turned to 270 degrees
- moved R4 0.10 mm to (106.2, 121.5)
- moved R7 0.10 mm to (109.5, 121.5)
Routing:
- net /DIM2: track 11.6 -> 18.7 mm
- net GND: track 33.2 -> 37.2 mm
- net /DIM1: track 16.4 -> 17.1 mm
Other:
- board text added: "VIN Max: 40V DC"
