File: LN2544_2ch_CWW.kicad_pcb (KiCad board)
At the start: 2 copper layers, 27 x 37 mm, 30 parts, among them P1 Vin, P2 LED, P3 DIM, P4 NTC, U1 LN2544, U2 LN2544

Commit message: PCB Update
Parts:
- removed R10, R3: 0R, Resistors_SMD:R_0805
- C3, C4: footprint Capacitors_SMD:C_1206 -> Capacitors_SMD:C_0805
- D1, D2: moved to F.Cu
- moved R4 22.0 mm to (106.2, 121.6), turned to 180 degrees
- moved R7 18.6 mm to (109.5, 121.6)
- moved R11 17.8 mm to (114.7, 121.6), turned to 180 degrees
- moved R13 15.0 mm to (102.4, 121.6), turned to 180 degrees
- moved R14 14.9 mm to (102.4, 119.3), turned to 0 degrees
- moved R15 14.7 mm to (102.4, 116.9), turned to 180 degrees
- moved R16 14.6 mm to (102.4, 114.6), turned to 0 degrees
- moved C1 12.7 mm to (112.4, 107.5), turned to 270 degrees
- moved C2 11.7 mm to (102.7, 107.4), turned to 270 degrees
- moved R6 10.8 mm to (117.9, 121.7)
- moved P3 10.5 mm to (119.0, 126.2)
- moved P1 8.74 mm to (104.7, 126.6), turned to 270 degrees
- moved R12 5.74 mm to (114.4, 109.9), turned to 90 degrees
- moved R5 5.43 mm to (104.7, 109.9), turned to 90 degrees
- moved D1 5.42 mm to (107.3, 106.5), turned to 0 degrees
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Connections:
- P3 pad 2: /DIM1 -> /DIM2
- P3 pad 3: /DIM2 -> /DIM1
- R6 pad 1: /DIM1 -> /DIM2
- R7 pad 1: /DIM2 -> /DIM1
Routing:
- net Net-(R5-Pad1): track 12.5 -> 0.00 mm
- net Net-(R12-Pad1): track 12.2 -> 2.75 mm
- net /NTC2: track 0.00 -> 6.63 mm
- net /CS1: track 4.78 -> 0.00 mm
- net GND: track 3.81 -> 7.58 mm
- net /VREF2: track 0.00 -> 2.62 mm
- net /V_IC: track 4.47 -> 2.08 mm
- net /DRAIN1: track 0.00 -> 0.95 mm
- net /CS2: track 4.72 -> 4.21 mm
- added copper zone on F.Cu, net /DRAIN1
Other:
- board size 27 x 37 mm -> 22 x 34 mm

Commit message: PCB UPDATE
Parts:
- added REF**111: Via_0406, BK_Common:Via_0406, F.Cu at (115.5, 116.3)
- added REF**111: Via_0406, BK_Common:Via_0406, F.Cu at (108.2, 116.5)
- added REF**111: Via_0406, BK_Common:Via_0406, F.Cu at (108.2, 115.2)
- added REF**111: Via_0406, BK_Common:Via_0406, F.Cu at (107.5, 115.2)
- added REF**111: Via_0406, BK_Common:Via_0406, F.Cu at (110.0, 110.0)
- added REF**111: Via_0406, BK_Common:Via_0406, F.Cu at (116.2, 116.2)
- added REF**111: Via_0406, BK_Common:Via_0406, F.Cu at (117.0, 116.2)
- added REF**111: Via_0406, BK_Common:Via_0406, F.Cu at (117.0, 115.0)
- added REF**111: Via_0406, BK_Common:Via_0406, F.Cu at (116.2, 115.0)
- added REF**111: Via_0406, BK_Common:Via_0406, F.Cu at (115.5, 115.0)
- added REF**111: Via_0406, BK_Common:Via_0406, F.Cu at (106.7, 115.2)
- added REF**111: Via_0406, BK_Common:Via_0406, F.Cu at (106.7, 116.5)
- added REF**111: Via_0406, BK_Common:Via_0406, F.Cu at (107.5, 116.5)
- added REF**11111: Via_0406, BK_Common:Via_0406, F.Cu at (119.7, 110.8)
- added REF**11121: Via_0406, BK_Common:Via_0406, F.Cu at (119.7, 110.0)
- added REF**11131: Via_0406, BK_Common:Via_0406, F.Cu at (119.7, 109.2)
- added REF**11141: Via_0406, BK_Common:Via_0406, F.Cu at (119.7, 108.4)
- added REF**11151: Via_0406, BK_Common:Via_0406, F.Cu at (119.7, 107.6)
- added REF**121: Via_0406, BK_Common:Via_0406, F.Cu at (110.0, 109.2)
- added REF**131: Via_0406, BK_Common:Via_0406, F.Cu at (110.0, 108.4)
- added REF**141: Via_0406, BK_Common:Via_0406, F.Cu at (110.0, 107.6)
- moved P3 0.84 mm to (119.8, 125.9)
- moved P1 0.70 mm to (104.7, 125.9)
Connections:
- U1 pad 9: (no net) -> GND
- U2 pad 9: (no net) -> GND
Routing:
- net VCC: track 0.00 -> 53.3 mm
- net /NTC1: track 0.00 -> 35.1 mm, vias 0 -> 2
- net GND: track 7.58 -> 38.1 mm, vias 0 -> 5
- net /NTC2: track 6.63 -> 27.2 mm
- net /DIM1: track 0.00 -> 16.2 mm
- net /V_IC: track 2.08 -> 17.3 mm
- net /LEDN2: track 0.00 -> 13.6 mm
- net /DIM2: track 0.00 -> 11.1 mm
- net /DRAIN1: track 0.95 -> 8.14 mm, vias 0 -> 1
- net /LEDN1: track 0.00 -> 6.69 mm
- net /DRAIN2: track 0.00 -> 4.55 mm
- net /CS1: track 0.00 -> 4.37 mm
- net Net-(R5-Pad1): track 0.00 -> 3.72 mm
- net /VREF1: track 0.00 -> 3.14 mm
- net Net-(R14-Pad2): track 0.00 -> 2.37 mm
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- added copper zone on F.Cu, net /DRAIN2
- added copper zone on B.Cu, net GND
Other:
- board size 22 x 34 mm -> 22 x 28 mm
- rule pad_to_mask_clearance: 0.2 -> 0
- board text added: "+"

Commit message: PCB UPdate
Parts:
- removed the REF**111 at (115.5, 116.3)
- removed the REF**111 at (108.2, 116.5)
- removed the REF**111 at (108.2, 115.2)
- removed the REF**111 at (107.5, 115.2)
- removed the REF**111 at (116.2, 116.2)
- removed the REF**111 at (117.0, 116.2)
- removed the REF**111 at (117.0, 115.0)
- removed the REF**111 at (116.2, 115.0)
- removed the REF**111 at (106.7, 115.2)
- removed the REF**111 at (106.7, 116.5)
- removed the REF**111 at (107.5, 116.5)
- added REF**: KiCAD Logo, Symbols:Symbol_KiCAD-Logo_CopperAndSilkScreenTop, B.Cu at (115.0, 113.8)
- added REF***: OSHW-Logo2_7.3x6mm_SilkScreen, Symbols:OSHW-Logo2_7.3x6mm_SilkScreen, B.Cu at (105.3, 114.3)
- added REF**111111: Via_0406, BK_Common:Via_0406, F.Cu at (106.7, 115.1)
- added REF**111112: Via_0406, BK_Common:Via_0406, F.Cu at (106.7, 116.6)
- added REF**111112: Via_0406, BK_Common:Via_0406, F.Cu at (115.4, 116.5)
- added REF**111121: Via_0406, BK_Common:Via_0406, F.Cu at (107.4, 115.1)
- added REF**111121: Via_0406, BK_Common:Via_0406, F.Cu at (116.1, 115.0)
- added REF**111122: Via_0406, BK_Common:Via_0406, F.Cu at (107.4, 116.6)
- added REF**111122: Via_0406, BK_Common:Via_0406, F.Cu at (116.1, 116.5)
- added REF**111131: Via_0406, BK_Common:Via_0406, F.Cu at (108.1, 115.1)
- added REF**111131: Via_0406, BK_Common:Via_0406, F.Cu at (116.8, 115.0)
- added REF**111132: Via_0406, BK_Common:Via_0406, F.Cu at (108.1, 116.6)
- added REF**111132: Via_0406, BK_Common:Via_0406, F.Cu at (116.8, 116.5)
- moved REF**111111 0.09 mm to (115.4, 115.0)
- renumbered REF**111 to REF**111111
Routing:
- net GND: track 38.1 -> 36.5 mm, vias 5 -> 7
Other:
- board text added: "1"
- board text added: "2"
- board text added: "DC Pow In"
- board text added: "Dim Input"
- board text added: "G"
- board text added: "LED Out"
- board text added: "LN2544_2ch_CWW V1.0"
- board text added: "LN2544_2ch_CWW V1.0 BK 2017"
- board text added: "NTC In"
- board text added: "Two channel LED Driver"

Commit message: Update
Parts:
- removed REF**: KiCAD Logo, Symbols:Symbol_KiCAD-Logo_CopperAndSilkScreenTop
- removed REF**111, REF**11111, REF**11121, REF**11131, REF**11141, REF**11151, REF**121, REF**131, REF**141: Via_0406, BK_Common:Via_0406
- added C5: 10n, Capacitors_SMD:C_0805, F.Cu at (117.6, 123.3)
- added C6: 10n, Capacitors_SMD:C_0805, F.Cu at (109.4, 123.4)
- added REF***: KiCad-Logo2_6mm_SilkScreen, Symbols:KiCad-Logo2_6mm_SilkScreen, B.Cu at (115.2, 114.9)
- moved REF*** 1.50 mm to (104.1, 115.1)
- moved R6 0.25 mm to (117.8, 121.4)
- moved P3 0.23 mm to (119.8, 126.1)
- moved R11 0.23 mm to (114.6, 121.4)
Connections:
- REF**111111 pad 1: GND -> /DRAIN1
- REF**111111 pad 1: GND -> /DRAIN2
- REF**111112 pad 1: GND -> /DRAIN1
- REF**111112 pad 1: GND -> /DRAIN2
- REF**111121 pad 1: GND -> /DRAIN1
- REF**111121 pad 1: GND -> /DRAIN2
- REF**111122 pad 1: GND -> /DRAIN1
- REF**111122 pad 1: GND -> /DRAIN2
- REF**111131 pad 1: GND -> /DRAIN1
- REF**111131 pad 1: GND -> /DRAIN2
- REF**111132 pad 1: GND -> /DRAIN1
- REF**111132 pad 1: GND -> /DRAIN2
- U1 pad 9: GND -> /DRAIN1
- U2 pad 9: GND -> /DRAIN2
Routing:
- net /DRAIN2: track 4.55 -> 27.8 mm
- net /DRAIN1: track 8.14 -> 22.9 mm, vias 1 -> 0
- net /V_IC: track 17.3 -> 22.5 mm
- net GND: track 36.5 -> 33.2 mm, vias 7 -> 9
- net /NTC1: track 35.1 -> 36.0 mm
- net /DIM2: track 11.1 -> 11.6 mm
Other:
- board text added: "DC In"
- board text removed: "DC Pow In"

Commit message: V1.1 Update
Parts:
- removed R2: R_CS12, Resistors_SMD:R_0805
- removed R9: R_CS22, Resistors_SMD:R_0805
- added C7: 1u/50V, Capacitors_SMD:C_1206, F.Cu at (101.8, 101.1)
- added C8: 1u/50V, Capacitors_SMD:C_1206, F.Cu at (111.7, 101.2)
- L1, L2: value 39uH -> 68uH; moved to F.Cu
- R1: value R_CS11 -> 1R5; footprint Resistors_SMD:R_0805 -> Resistors_SMD:R_1210
- R11: value RNTC2 -> 24k
- R12: value RO2 -> 24k
- R4: value RNTC1 -> 24k
- R5: value RO1 -> 24k
- R6, R7: value 10K -> 62k
- R8: value R_CS21 -> 1R5; footprint Resistors_SMD:R_0805 -> Resistors_SMD:R_1210
- moved REF*** 14.2 mm to (111.0, 102.7)
- moved REF*** 7.00 mm to (110.9, 109.4)
- moved L2 6.67 mm to (116.1, 101.8)
- moved L1 6.63 mm to (106.3, 101.9)
- moved P2 5.23 mm to (101.9, 96.9)
- moved P4 5.08 mm to (115.1, 96.9)
- moved R8 1.30 mm to (117.6, 109.9), turned to 180 degrees
- moved R1 0.66 mm to (107.8, 109.9), turned to 180 degrees
Routing:
- net /DRAIN2: track 27.8 -> 38.9 mm
- net VCC: track 53.3 -> 64.0 mm, vias 0 -> 4
- net /DRAIN1: track 22.9 -> 29.9 mm
- net /NTC2: track 27.3 -> 32.3 mm, vias 0 -> 1
- net GND: track 33.2 -> 28.4 mm
- net /NTC1: track 36.0 -> 40.0 mm, vias 2 -> 1
- net /LEDN2: track 13.6 -> 10.4 mm
- net /LEDN1: track 6.69 -> 9.35 mm
- net /CS1: track 4.37 -> 3.77 mm
- net /CS2: track 4.21 -> 4.76 mm
Other:
- board size 22 x 28 mm -> 22 x 33 mm
- board text added: "LN2544_2ch_CWW V1.1"
- board text added: "LN2544_2ch_CWW V1.1 BK 2017"
- board text removed: "LN2544_2ch_CWW V1.0"
- board text removed: "LN2544_2ch_CWW V1.0 BK 2017"
