File: LN2544_2ch_CWW.sch (KiCad schematic (older format))
At the start: 30 parts, among them P1 Vin, P2 LED, P3 DIM, P4 NTC, U1 LN2544, U2 LN2544

Commit message: Upd
Parts:
- R11: value RNTC2 -> 12K
- R2: value R_CS12 -> 1.4R
- R4: value RNTC1 -> 12K
- R9: value R_CS22 -> 1.4R
Other:
- note added: "If R6,R7 populated, default LED off."
- note added: "NTC 10K Vref=1.2V Regulation 0.05V<VNTC<0.25V\nWith RNTC 12.6K starts correcting at 55C\nreaches 0A at 100C"
- note added: "RCS=0.5/IledPeak\nRCS=0.5/0.350=1.4R\nPCS=0.350**1.4=0.17W"
Changed lines of the file:
@@
 LIBS:contrib
 LIBS:valves
-LIBS:BK_Common
-LIBS:BK_LED_Drivers
 LIBS:LN2544_2ch_CWW-cache
 EELAYER 25 0
@@
 P 8300 5300
 F 0 "R9" H 8330 5320 50  0000 L CNN
-F 1 "R_CS22" H 8330 5260 50  0000 L CNN
+F 1 "1.4R" H 8330 5260 50  0000 L CNN
 F 2 "Resistors_SMD:R_0805" H 8350 5150 50  0001 C CNN
 F 3 "" H 8300 5300 50  0000 C CNN
@@
 P 6550 5600
 F 0 "R11" H 6580 5620 50  0000 L CNN
-F 1 "RNTC2" H 6580 5560 50  0000 L CNN
+F 1 "12K" H 6580 5560 50  0000 L CNN
 F 2 "Resistors_SMD:R_0805" H 6600 5450 50  0001 C CNN
 F 3 "" H 6550 5600 50  0000 C CNN
@@
 P 8500 2750
 F 0 "R2" H 8530 2770 50  0000 L CNN
-F 1 "R_CS12" H 8530 2710 50  0000 L CNN
+F 1 "1.4R" H 8530 2710 50  0000 L CNN
 F 2 "Resistors_SMD:R_0805" H 8550 2600 50  0001 C CNN
 F 3 "" H 8500 2750 50  0000 C CNN
@@
 P 6750 3050
 F 0 "R4" H 6780 3070 50  0000 L CNN
-F 1 "RNTC1" H 6780 3010 50  0000 L CNN
+F 1 "12K" H 6780 3010 50  0000 L CNN
 F 2 "Resistors_SMD:R_0805" H 6800 2900 50  0001 C CNN
 F 3 "" H 6750 3050 50  0000 C CNN
@@
 	8150 4950 8150 4850
 Connection ~ 8150 4850
+Text Notes 4500 6850 0    60   ~ 0
+NTC 10K Vref=1.2V Regulation 0.05V<VNTC<0.25V\nWith RNTC 12.6K starts correcting at 55C\nreaches 0A at 100C
+Text Notes 9000 5400 0    60   ~ 0
+RCS=0.5/IledPeak\nRCS=0.5/0.350=1.4R\nPCS=0.350**1.4=0.17W
+Text Notes 2050 3050 0    60   ~ 0
+If R6,R7 populated, default LED off.
 $EndSCHEMATC
