File: LN2544_2ch_CWW.sch (KiCad schematic (older format))
At the start: 30 parts, among them P1 Vin, P2 LED, P3 DIM, P4 NTC, U1 LN2544, U2 LN2544

Commit message: Update
Parts:
- removed R10, R3: 0R, Resistors_SMD:R_0805, symbol R_SMD_0805
- added C5, C6: 10n, Capacitors_SMD:C_0805, symbol C_Cer_SMD_0805
- C3, C4: footprint Capacitors_SMD:C_1206 -> Capacitors_SMD:C_0805
Connections:
- wire segments 86 -> 90
Other:
- moved on the sheet: R7
Changed lines of the file:
@@
 LIBS:BK_Common
 LIBS:BK_LED_Drivers
+LIBS:LN2544_2ch_CWW-cache
 EELAYER 25 0
 EELAYER END
@@
 F 0 "C4" H 8010 4270 50  0000 L CNN
 F 1 "10uF/16V" H 8010 4120 50  0000 L CNN
-F 2 "Capacitors_SMD:C_1206" H 8000 4050 50  0001 C CNN
+F 2 "Capacitors_SMD:C_0805" H 8000 4050 50  0001 C CNN
 F 3 "" H 8000 4200 50  0000 C CNN
 	1    8000 4200
@@
 	1    0    0    -1
 $EndComp
+Text Label 1700 3150 0    60   ~ 0
+DIM1
 Text Label 1700 3250 0    60   ~ 0
-DIM1
-Text Label 1700 3150 0    60   ~ 0
 DIM2
 Text Label 1700 2250 0    60   ~ 0
@@
 	1    0    0    -1
 $EndComp
-$Comp
-L R_SMD_0805 R10
-U 1 1 59461051
-P 6250 5600
-F 0 "R10" H 6280 5620 50  0000 L CNN
-F 1 "0R" H 6280 5560 50  0000 L CNN
-F 2 "Resistors_SMD:R_0805" H 6300 5450 50  0001 C CNN
-F 3 "" H 6250 5600 50  0000 C CNN
-	1    6250 5600
-	1    0    0    -1
-$EndComp
 Text Label 6400 4950 0    60   ~ 0
 VREF2
 Text Label 6400 5050 0    60   ~ 0
 NTC2
-$Comp
-L GND #PWR09
-U 1 1 594616EA
-P 6250 5800
-F 0 "#PWR09" H 6250 5550 50  0001 C CNN
-F 1 "GND" H 6250 5650 50  0000 C CNN
-F 2 "" H 6250 5800 50  0000 C CNN
-F 3 "" H 6250 5800 50  0000 C CNN
-	1    6250 5800
-	1    0    0    -1
-$EndComp
 Text Label 6600 5950 0    60   ~ 0
 VREF2
@@
 L R_SMD_0805 R7
 U 1 1 59462418
-P 2450 3450
-F 0 "R7" H 2480 3470 50  0000 L CNN
-F 1 "10K" H 2480 3410 50  0000 L CNN
-F 2 "Resistors_SMD:R_0805" H 2500 3300 50  0001 C CNN
-F 3 "" H 2450 3450 50  0000 C CNN
-	1    2450 3450
+P 2900 3450
+F 0 "R7" H 2930 3470 50  0000 L CNN
+F 1 "10K" H 2930 3410 50  0000 L CNN
+F 2 "Resistors_SMD:R_0805" H 2950 3300 50  0001 C CNN
+F 3 "" H 2900 3450 50  0000 C CNN
+	1    2900 3450
 	1    0    0    -1
 $EndComp
@@
 	1700 3350 1700 3450
 Wire Wire Line
-	1650 3250 2200 3250
-Wire Wire Line
-	1650 3150 2450 3150
+	1650 3250 2450 3250
+Wire Wire Line
+	1650 3150 3150 3150
 Wire Wire Line
 	1650 2350 2150 2350
@@
 Connection ~ 8000 4000
 Wire Wire Line
-	6250 5050 6850 5050
-Wire Wire Line
 	6850 4950 6400 4950
 Wire Wire Line
@@
 Wire Wire Line
 	6550 5950 6900 5950
-Wire Wire Line
-	6250 5050 6250 5500
 Wire Wire Line
 	6550 5500 6550 5050
 Connection ~ 6550 5050
 Wire Wire Line
-	6250 5700 6250 5800
-Wire Wire Line
-	2450 3150 2450 3350
-Wire Wire Line
 	2200 3250 2200 3350
 Wire Wire Line
 	2200 3550 2200 3650
 Wire Wire Line
-	2200 3650 2450 3650
-Wire Wire Line
-	2450 3650 2450 3550
-$Comp
-L GND #PWR010
+	2200 3650 3150 3650
+$Comp
+L GND #PWR09
 U 1 1 59462703
 P 2300 3700
-F 0 "#PWR010" H 2300 3450 50  0001 C CNN
+F 0 "#PWR09" H 2300 3450 50  0001 C CNN
 F 1 "GND" H 2300 3550 50  0000 C CNN
 F 2 "" H 2300 3700 50  0000 C CNN
@@
 F 0 "C3" H 8210 1720 50  0000 L CNN
 F 1 "10uF/16V" H 8210 1570 50  0000 L CNN
-F 2 "Capacitors_SMD:C_1206" H 8200 1500 50  0001 C CNN
+F 2 "Capacitors_SMD:C_0805" H 8200 1500 50  0001 C CNN
 F 3 "" H 8200 1650 50  0000 C CNN
 	1    8200 1650
@@
 $EndComp
 $Comp
-L GND #PWR011
+L GND #PWR010
 U 1 1 59463A0D
 P 8300 3350
-F 0 "#PWR011" H 8300 3100 50  0001 C CNN
+F 0 "#PWR010" H 8300 3100 50  0001 C CNN
 F 1 "GND" H 8300 3200 50  0000 C CNN
 F 2 "" H 8300 3350 50  0000 C CNN
@@
 LEDN1
 $Comp
-L VCC #PWR012
+L VCC #PWR011
 U 1 1 59463A14
 P 8850 1800
-F 0 "#PWR012" H 8850 1650 50  0001 C CNN
+F 0 "#PWR011" H 8850 1650 50  0001 C CNN
 F 1 "VCC" H 8850 1950 50  0000 C CNN
 F 2 "" H 8850 1800 50  0000 C CNN
@@
 $EndComp
 $Comp
-L GND #PWR013
+L GND #PWR012
 U 1 1 59463A1A
 P 8200 1850
-F 0 "#PWR013" H 8200 1600 50  0001 C CNN
+F 0 "#PWR012" H 8200 1600 50  0001 C CNN
 F 1 "GND" H 8200 1700 50  0000 C CNN
 F 2 "" H 8200 1850 50  0000 C CNN
@@
 	1    0    0    -1
 $EndComp
-$Comp
-L R_SMD_0805 R3
-U 1 1 59463A27
-P 6450 3050
-F 0 "R3" H 6480 3070 50  0000 L CNN
-F 1 "0R" H 6480 3010 50  0000 L CNN
-F 2 "Resistors_SMD:R_0805" H 6500 2900 50  0001 C CNN
-F 3 "" H 6450 3050 50  0000 C CNN
-	1    6450 3050
-	1    0    0    -1
-$EndComp
 Text Label 6600 2400 0    60   ~ 0
 VREF1
 Text Label 6600 2500 0    60   ~ 0
 NTC1
-$Comp
-L GND #PWR014
-U 1 1 59463A2F
-P 6450 3250
-F 0 "#PWR014" H 6450 3000 50  0001 C CNN
-F 1 "GND" H 6450 3100 50  0000 C CNN
-F 2 "" H 6450 3250 50  0000 C CNN
-F 3 "" H 6450 3250 50  0000 C CNN
-	1    6450 3250
-	1    0    0    -1
-$EndComp
 Text Label 6800 3400 0    60   ~ 0
 VREF1
@@
 Connection ~ 8200 1450
 Wire Wire Line
-	6450 2500 7050 2500
-Wire Wire Line
 	7050 2400 6600 2400
 Wire Wire Line
@@
 Wire Wire Line
 	6750 3400 7100 3400
-Wire Wire Line
-	6450 2500 6450 2950
 Wire Wire Line
 	6750 2950 6750 2500
 Connection ~ 6750 2500
-Wire Wire Line
-	6450 3150 6450 3250
 $Comp
 L C_Cer_SMD_1206 C1
@@
 	4450 1250 4450 1400
 $Comp
-L VCC #PWR015
+L VCC #PWR013
 U 1 1 5946BEF7
 P 4150 1150
-F 0 "#PWR015" H 4150 1000 50  0001 C CNN
+F 0 "#PWR013" H 4150 1000 50  0001 C CNN
 F 1 "VCC" H 4150 1300 50  0000 C CNN
 F 2 "" H 4150 1150 50  0000 C CNN
@@
 $EndComp
 $Comp
-L GND #PWR016
+L GND #PWR014
 U 1 1 5946BF7A
 P 4150 1850
-F 0 "#PWR016" H 4150 1600 50  0001 C CNN
+F 0 "#PWR014" H 4150 1600 50  0001 C CNN
 F 1 "GND" H 4150 1700 50  0000 C CNN
 F 2 "" H 4150 1850 50  0000 C CNN
@@
 Connection ~ 4150 1250
 $Comp
-L VCC #PWR017
+L VCC #PWR015
 U 1 1 59470E5E
 P 2150 2300
-F 0 "#PWR017" H 2150 2150 50  0001 C CNN
+F 0 "#PWR015" H 2150 2150 50  0001 C CNN
 F 1 "VCC" H 2150 2450 50  0000 C CNN
 F 2 "" H 2150 2300 50  0000 C CNN
@@
 Text Label 8050 5050 0    60   ~ 0
 CS2
+Wire Wire Line
+	7050 2500 6600 2500
+Wire Wire Line
+	6850 5050 6400 5050
+$Comp
+L C_Cer_SMD_0805 C5
+U 1 1 594B2C4B
+P 2450 3450
+F 0 "C5" H 2460 3520 50  0000 L CNN
+F 1 "10n" H 2460 3370 50  0000 L CNN
+F 2 "Capacitors_SMD:C_0805" H 2450 3300 50  0001 C CNN
+F 3 "" H 2450 3450 50  0000 C CNN
+	1    2450 3450
+	1    0    0    -1
+$EndComp
+$Comp
+L C_Cer_SMD_0805 C6
+U 1 1 594B2EB7
+P 3150 3450
+F 0 "C6" H 3160 3520 50  0000 L CNN
+F 1 "10n" H 3160 3370 50  0000 L CNN
+F 2 "Capacitors_SMD:C_0805" H 3150 3300 50  0001 C CNN
+F 3 "" H 3150 3450 50  0000 C CNN
+	1    3150 3450
+	1    0    0    -1
+$EndComp
+Wire Wire Line
+	3150 3150 3150 3350
+Wire Wire Line
+	2900 3350 2900 3150
+Connection ~ 2900 3150
+Wire Wire Line
+	2450 3250 2450 3350
+Connection ~ 2200 3250
+Wire Wire Line
+	3150 3650 3150 3550
+Wire Wire Line
+	2900 3550 2900 3650
+Connection ~ 2900 3650
+Wire Wire Line
+	2450 3550 2450 3650
+Connection ~ 2450 3650
+Wire Wire Line
+	8250 2400 8300 2400
+Wire Wire Line
+	8300 2400 8300 2300
+Connection ~ 8300 2300
+Wire Wire Line
+	8050 4950 8150 4950
+Wire Wire Line
+	8150 4950 8150 4850
+Connection ~ 8150 4850
 $EndSCHEMATC

Commit message: V1.1 Update
Parts:
- removed R2: R_CS12, Resistors_SMD:R_0805, symbol R_SMD_0805
- removed R9: R_CS22, Resistors_SMD:R_0805, symbol R_SMD_0805
- added C7, C8: 1u/50V, Capacitors_SMD:C_1206, symbol C_Cer_SMD_1206
- L1, L2: value 39uH -> 68uH
- R1: value R_CS11 -> 1R5; footprint Resistors_SMD:R_0805 -> Resistors_SMD:R_1210
- R11: value RNTC2 -> 24k
- R12: value RO2 -> 24k
- R4: value RNTC1 -> 24k
- R5: value RO1 -> 24k
- R6, R7: value 10K -> 62k
- R8: value R_CS21 -> 1R5; footprint Resistors_SMD:R_0805 -> Resistors_SMD:R_1210
Other:
- note added: "62K pull-down: without pwm input \nit will run at about 30% current\nif not used it will run at 100% current\nwithout input"
- note added: "Below 300mA L1, L2 can be increased to 100uH"
- note added: "C7,C8 Optional"
- note added: "Common positive LED \ndriver outputs"
- note added: "Iled = 0.5V/RCS"
- note added: "Iled = 0.5V/RCS\nIled = 0.5/1.5 = 333mA\nPcs = 333mA*333mA*1.5 = 0.166W"
- note added: "Maximum input voltage: 36V DC\nNo input protection for efficiency"
- note added: "NTC optional: 10K NTC mounted on LED\nCurrent decreased from about 50C\nCurrent goes to 0 at about 90C"
- moved on the sheet: C1, C2
Changed lines of the file:
@@
 encoding utf-8
 Sheet 1 1
-Title ""
-Date ""
-Rev ""
-Comp ""
+Title "LN2544 2 Channel Common Positive  LED Driver"
+Date "2017-11-12"
+Rev "V1.1"
+Comp "BK"
 Comment1 ""
 Comment2 ""
@@
 P 8900 4850
 F 0 "L2" H 8930 4890 50  0000 L CNN
-F 1 "39uH" H 8930 4810 50  0000 L CNN
+F 1 "68uH" H 8930 4810 50  0000 L CNN
 F 2 "BK_Common:IND_SMD_CD54" H 8900 4850 50  0001 C CNN
 F 3 "" H 8900 4850 50  0000 C CNN
@@
 P 8100 5300
 F 0 "R8" H 8130 5320 50  0000 L CNN
-F 1 "R_CS21" H 7800 5250 50  0000 L CNN
-F 2 "Resistors_SMD:R_0805" H 8150 5150 50  0001 C CNN
+F 1 "1R5" H 7875 5275 50  0000 L CNN
+F 2 "Resistors_SMD:R_1210" H 8150 5150 50  0001 C CNN
 F 3 "" H 8100 5300 50  0000 C CNN
 	1    8100 5300
-	1    0    0    -1
-$EndComp
-$Comp
-L R_SMD_0805 R9
-U 1 1 5945E4A8
-P 8300 5300
-F 0 "R9" H 8330 5320 50  0000 L CNN
-F 1 "R_CS22" H 8330 5260 50  0000 L CNN
-F 2 "Resistors_SMD:R_0805" H 8350 5150 50  0001 C CNN
-F 3 "" H 8300 5300 50  0000 C CNN
-	1    8300 5300
 	1    0    0    -1
 $EndComp
@@
 P 7350 5600
 F 0 "R12" H 7380 5620 50  0000 L CNN
-F 1 "RO2" H 7380 5560 50  0000 L CNN
+F 1 "24k" H 7380 5560 50  0000 L CNN
 F 2 "Resistors_SMD:R_0805" H 7400 5450 50  0001 C CNN
 F 3 "" H 7350 5600 50  0000 C CNN
@@
 Text Label 1700 6750 0    60   ~ 0
 V_IC
-Text Label 9200 4850 0    60   ~ 0
+Text Label 9125 4850 0    60   ~ 0
 LEDN2
 $Comp
@@
 P 6550 5600
 F 0 "R11" H 6580 5620 50  0000 L CNN
-F 1 "RNTC2" H 6580 5560 50  0000 L CNN
+F 1 "24k" H 6580 5560 50  0000 L CNN
 F 2 "Resistors_SMD:R_0805" H 6600 5450 50  0001 C CNN
 F 3 "" H 6550 5600 50  0000 C CNN
@@
 P 2200 3450
 F 0 "R6" H 2230 3470 50  0000 L CNN
-F 1 "10K" H 2230 3410 50  0000 L CNN
+F 1 "62k" H 2230 3410 50  0000 L CNN
 F 2 "Resistors_SMD:R_0805" H 2250 3300 50  0001 C CNN
 F 3 "" H 2200 3450 50  0000 C CNN
@@
 P 2900 3450
 F 0 "R7" H 2930 3470 50  0000 L CNN
-F 1 "10K" H 2930 3410 50  0000 L CNN
+F 1 "62k" H 2930 3410 50  0000 L CNN
 F 2 "Resistors_SMD:R_0805" H 2950 3300 50  0001 C CNN
 F 3 "" H 2900 3450 50  0000 C CNN
@@
 	7350 5700 7350 5800
 Wire Wire Line
-	7350 5800 8300 5800
-Wire Wire Line
-	8300 5800 8300 5400
-Wire Wire Line
 	8100 5400 8100 5900
 Connection ~ 8100 5800
 Wire Wire Line
 	8100 5200 8100 5050
-Wire Wire Line
-	8050 5050 8300 5050
-Wire Wire Line
-	8300 5050 8300 5200
-Connection ~ 8100 5050
 Wire Wire Line
 	1650 4250 1700 4250
@@
 P 9100 2300
 F 0 "L1" H 9130 2340 50  0000 L CNN
-F 1 "39uH" H 9130 2260 50  0000 L CNN
+F 1 "68uH" H 9130 2260 50  0000 L CNN
 F 2 "BK_Common:IND_SMD_CD54" H 9100 2300 50  0001 C CNN
 F 3 "" H 9100 2300 50  0000 C CNN
@@
 P 8300 2750
 F 0 "R1" H 8330 2770 50  0000 L CNN
-F 1 "R_CS11" H 8000 2700 50  0000 L CNN
-F 2 "Resistors_SMD:R_0805" H 8350 2600 50  0001 C CNN
+F 1 "1R5" H 8075 2725 50  0000 L CNN
+F 2 "Resistors_SMD:R_1210" H 8350 2600 50  0001 C CNN
 F 3 "" H 8300 2750 50  0000 C CNN
 	1    8300 2750
-	1    0    0    -1
-$EndComp
-$Comp
-L R_SMD_0805 R2
-U 1 1 59463A01
-P 8500 2750
-F 0 "R2" H 8530 2770 50  0000 L CNN
-F 1 "R_CS12" H 8530 2710 50  0000 L CNN
-F 2 "Resistors_SMD:R_0805" H 8550 2600 50  0001 C CNN
-F 3 "" H 8500 2750 50  0000 C CNN
-	1    8500 2750
 	1    0    0    -1
 $EndComp
@@
 P 7550 3050
 F 0 "R5" H 7580 3070 50  0000 L CNN
-F 1 "RO1" H 7580 3010 50  0000 L CNN
+F 1 "24k" H 7580 3010 50  0000 L CNN
 F 2 "Resistors_SMD:R_0805" H 7600 2900 50  0001 C CNN
 F 3 "" H 7550 3050 50  0000 C CNN
@@
 P 6750 3050
 F 0 "R4" H 6780 3070 50  0000 L CNN
-F 1 "RNTC1" H 6780 3010 50  0000 L CNN
+F 1 "24k" H 6780 3010 50  0000 L CNN
 F 2 "Resistors_SMD:R_0805" H 6800 2900 50  0001 C CNN
 F 3 "" H 6750 3050 50  0000 C CNN
@@
 	7550 3150 7550 3250
 Wire Wire Line
-	7550 3250 8500 3250
-Wire Wire Line
-	8500 3250 8500 2850
-Wire Wire Line
 	8300 2850 8300 3350
 Connection ~ 8300 3250
@@
 	8300 2650 8300 2500
 Wire Wire Line
-	8250 2500 8500 2500
-Wire Wire Line
-	8500 2500 8500 2650
-Connection ~ 8300 2500
-Wire Wire Line
 	8250 2300 9000 2300
 Wire Wire Line
@@
 L C_Cer_SMD_1206 C1
 U 1 1 5946BA06
-P 3900 1500
-F 0 "C1" H 3910 1570 50  0000 L CNN
-F 1 "10uF/50V" H 3910 1420 50  0000 L CNN
-F 2 "Capacitors_SMD:C_1206" H 3900 1350 50  0001 C CNN
-F 3 "" H 3900 1500 50  0000 C CNN
-	1    3900 1500
+P 2825 6050
+F 0 "C1" H 2835 6120 50  0000 L CNN
+F 1 "10uF/50V" H 2835 5970 50  0000 L CNN
+F 2 "Capacitors_SMD:C_1206" H 2825 5900 50  0001 C CNN
+F 3 "" H 2825 6050 50  0000 C CNN
+	1    2825 6050
 	1    0    0    -1
 $EndComp
@@
 L C_Cer_SMD_1206 C2
 U 1 1 5946BC56
-P 4450 1500
-F 0 "C2" H 4460 1570 50  0000 L CNN
-F 1 "10uF/50V" H 4460 1420 50  0000 L CNN
-F 2 "Capacitors_SMD:C_1206" H 4450 1350 50  0001 C CNN
-F 3 "" H 4450 1500 50  0000 C CNN
-	1    4450 1500
-	1    0    0    -1
-$EndComp
-Wire Wire Line
-	3900 1600 3900 1750
-Wire Wire Line
-	3900 1750 4450 1750
-Wire Wire Line
-	4450 1750 4450 1600
-Wire Wire Line
-	3900 1400 3900 1250
-Wire Wire Line
-	3900 1250 4450 1250
-Wire Wire Line
-	4450 1250 4450 1400
+P 3375 6050
+F 0 "C2" H 3385 6120 50  0000 L CNN
+F 1 "10uF/50V" H 3385 5970 50  0000 L CNN
+F 2 "Capacitors_SMD:C_1206" H 3375 5900 50  0001 C CNN
+F 3 "" H 3375 6050 50  0000 C CNN
+	1    3375 6050
+	1    0    0    -1
+$EndComp
+Wire Wire Line
+	2825 6150 2825 6300
+Wire Wire Line
+	2825 6300 3375 6300
+Wire Wire Line
+	3375 6300 3375 6150
+Wire Wire Line
+	2825 5950 2825 5800
+Wire Wire Line
+	2825 5800 3375 5800
+Wire Wire Line
+	3375 5800 3375 5950
 $Comp
 L VCC #PWR013
 U 1 1 5946BEF7
-P 4150 1150
-F 0 "#PWR013" H 4150 1000 50  0001 C CNN
-F 1 "VCC" H 4150 1300 50  0000 C CNN
-F 2 "" H 4150 1150 50  0000 C CNN
-F 3 "" H 4150 1150 50  0000 C CNN
-	1    4150 1150
+P 3075 5700
+F 0 "#PWR013" H 3075 5550 50  0001 C CNN
+F 1 "VCC" H 3075 5850 50  0000 C CNN
+F 2 "" H 3075 5700 50  0000 C CNN
+F 3 "" H 3075 5700 50  0000 C CNN
+	1    3075 5700
 	1    0    0    -1
 $EndComp
@@
 L GND #PWR014
 U 1 1 5946BF7A
-P 4150 1850
-F 0 "#PWR014" H 4150 1600 50  0001 C CNN
-F 1 "GND" H 4150 1700 50  0000 C CNN
-F 2 "" H 4150 1850 50  0000 C CNN
-F 3 "" H 4150 1850 50  0000 C CNN
-	1    4150 1850
-	1    0    0    -1
-$EndComp
-Wire Wire Line
-	4150 1850 4150 1750
-Connection ~ 4150 1750
-Wire Wire Line
-	4150 1150 4150 1250
-Connection ~ 4150 1250
+P 3075 6400
+F 0 "#PWR014" H 3075 6150 50  0001 C CNN
+F 1 "GND" H 3075 6250 50  0000 C CNN
+F 2 "" H 3075 6400 50  0000 C CNN
+F 3 "" H 3075 6400 50  0000 C CNN
+	1    3075 6400
+	1    0    0    -1
+$EndComp
+Wire Wire Line
+	3075 6400 3075 6300
+Connection ~ 3075 6300
+Wire Wire Line
+	3075 5700 3075 5800
+Connection ~ 3075 5800
 $Comp
 L VCC #PWR015
@@
 Text Label 8250 2500 0    60   ~ 0
 CS1
-Text Label 8050 5050 0    60   ~ 0
-CS2
 Wire Wire Line
 	7050 2500 6600 2500
@@
 	8150 4950 8150 4850
 Connection ~ 8150 4850
+Wire Wire Line
+	7350 5800 8100 5800
+Wire Wire Line
+	8100 5050 8050 5050
+Text Label 8050 5050 0    60   ~ 0
+CS2
+Wire Wire Line
+	8300 2500 8250 2500
+Wire Wire Line
+	7550 3250 8300 3250
+$Comp
+L C_Cer_SMD_1206 C8
+U 1 1 5A068E9D
+P 9450 4600
+F 0 "C8" H 9460 4670 50  0000 L CNN
+F 1 "1u/50V" H 9460 4520 50  0000 L CNN
+F 2 "Capacitors_SMD:C_1206" H 9450 4450 50  0001 C CNN
+F 3 "" H 9450 4600 50  0000 C CNN
+	1    9450 4600
+	1    0    0    -1
+$EndComp
+$Comp
+L VCC #PWR016
+U 1 1 5A068FE2
+P 9450 4350
+F 0 "#PWR016" H 9450 4200 50  0001 C CNN
+F 1 "VCC" H 9450 4500 50  0000 C CNN
+F 2 "" H 9450 4350 50  0000 C CNN
+F 3 "" H 9450 4350 50  0000 C CNN
+	1    9450 4350
+	1    0    0    -1
+$EndComp
+Wire Wire Line
+	9450 4350 9450 4500
+Wire Wire Line
+	9450 4850 9450 4700
+$Comp
+L C_Cer_SMD_1206 C7
+U 1 1 5A06925E
+P 9650 2075
+F 0 "C7" H 9660 2145 50  0000 L CNN
+F 1 "1u/50V" H 9660 1995 50  0000 L CNN
+F 2 "Capacitors_SMD:C_1206" H 9650 1925 50  0001 C CNN
+F 3 "" H 9650 2075 50  0000 C CNN
+	1    9650 2075
+	1    0    0    -1
+$EndComp
+$Comp
+L VCC #PWR017
+U 1 1 5A06949A
+P 9650 1800
+F 0 "#PWR017" H 9650 1650 50  0001 C CNN
+F 1 "VCC" H 9650 1950 50  0000 C CNN
+F 2 "" H 9650 1800 50  0000 C CNN
+F 3 "" H 9650 1800 50  0000 C CNN
+	1    9650 1800
+	1    0    0    -1
+$EndComp
+Wire Wire Line
+	9650 1800 9650 1975
+Wire Wire Line
+	9650 2300 9650 2175
+Text Notes 8450 2775 0    60   ~ 12
+Iled = 0.5V/RCS
+Text Notes 8275 5425 0    60   ~ 12
+Iled = 0.5V/RCS\nIled = 0.5/1.5 = 333mA\nPcs = 333mA*333mA*1.5 = 0.166W
+Text Notes 9525 4425 0    60   ~ 12
+C7,C8 Optional
+Text Notes 9700 1925 0    60   ~ 12
+C7,C8 Optional
+Text Notes 3400 3575 0    60   ~ 12
+62K pull-down: without pwm input \nit will run at about 30% current\nif not used it will run at 100% current\nwithout input
+Text Notes 2325 2275 0    60   ~ 12
+Common positive LED \ndriver outputs
+Text Notes 2025 4300 0    60   ~ 12
+NTC optional: 10K NTC mounted on LED\nCurrent decreased from about 50C\nCurrent goes to 0 at about 90C
+Text Notes 1875 1300 0    60   ~ 12
+Maximum input voltage: 36V DC\nNo input protection for efficiency
+Text Notes 8275 5650 0    60   ~ 12
+Below 300mA L1, L2 can be increased to 100uH
 $EndSCHEMATC
